File: corne-chocolate/pcb/corne-chocolate.kicad_pcb (KiCad board)
At the start: 2 copper layers, 133.8 x 91.4 mm, 98 parts, among them J3 LED, P1 i2c-pin, P2 i2c-pin, SW1 SW_PUSH, SW10 SW_PUSH, SW11 SW_PUSH, SW12 SW_PUSH, SW13 SW_PUSH, SW14 SW_PUSH, SW15 SW_PUSH, SW16 SW_PUSH, SW17 SW_PUSH, SW18 SW_PUSH, SW19 SW_PUSH, SW2 SW_PUSH, SW20 SW_PUSH, SW21 SW_PUSH, SW3 SW_PUSH, SW4 SW_PUSH, SW5 SW_PUSH, SW6 SW_PUSH, SW7 SW_PUSH, SW8 SW_PUSH, SW9 SW_PUSH, U1 ProMicro

Commit message: squash!  moved v3 to choc
foostan does not distinguish versions by subdirectory (see eg. kicad6_corne_cherry). Also it messes up kicad libraries

Note: This would undo #165, supposedly done onto chocolate v2?
Parts:
- removed ? (x9): , kbd:LEGO_HOLE
- removed the G*** at (184.0, 85.0)
- removed the G*** at (184.7, 85.2)
- removed JP2, JP3, JP4, JP5, JP6, JP7, JP8, JP9: , kbd:Jumper
- removed L1, L10, L11, L12, L13, L14, L15, L16, L17, L18, L19, L2, L20, L21, L3, L4, L5, L6, L7, L8, L9: SK6812MINI, kbd:SK6812MINI_rev
- removed L22, L23, L24, L25, L26, L27: SK6812MINI, kbd:SK6812MINI_underglow_rev
- removed OLED: OLED, kbd:OLED
- removed P1, P2: i2c-pin, kbd:1pin_conn
- removed R1, R2: R, kbd:R
- removed TRRS: MJ-4PP-9, kbd:MJ-4PP-9
- removed data: , kbd:JPC2
- added D22: D, kbd:D3_SMD_v2, B.Cu at (284.2, 35.8)
- added D23: D, kbd:D3_SMD_v2, B.Cu at (265.2, 35.8)
- added D24: D, kbd:D3_SMD_v2, B.Cu at (246.2, 31.0)
- added D25: D, kbd:D3_SMD_v2, B.Cu at (227.2, 28.6)
- added D26: D, kbd:D3_SMD_v2, B.Cu at (208.2, 31.0)
- added D27: D, kbd:D3_SMD_v2, B.Cu at (189.2, 33.4)
- added D28: D, kbd:D3_SMD_v2, B.Cu at (284.2, 54.6)
- added D29: D, kbd:D3_SMD_v2, B.Cu at (265.2, 54.8)
- added D30: D, kbd:D3_SMD_v2, B.Cu at (246.2, 50.0)
- added D31: D, kbd:D3_SMD_v2, B.Cu at (227.2, 47.6)
- added D32: D, kbd:D3_SMD_v2, B.Cu at (208.2, 50.0)
- added D33: D, kbd:D3_SMD_v2, B.Cu at (189.2, 52.4)
- added D34: D, kbd:D3_SMD_v2, B.Cu at (284.2, 73.8)
- added D35: D, kbd:D3_SMD_v2, B.Cu at (265.2, 73.8)
- added D36: D, kbd:D3_SMD_v2, B.Cu at (246.2, 69.0)
- added D37: D, kbd:D3_SMD_v2, B.Cu at (227.2, 66.7)
- added D38: D, kbd:D3_SMD_v2, B.Cu at (208.2, 69.0)
- added D39: D, kbd:D3_SMD_v2, B.Cu at (189.2, 71.4)
- added D40: D, kbd:D3_SMD_v2, B.Cu at (217.7, 88.6)
- added D41: D, kbd:D3_SMD_v2, B.Cu at (199.6, 87.9)
- added D42: D, kbd:D3_SMD_v2, B.Cu at (196.8, 87.9)
- added G***: LOGO, kbd:corne-logo-horizontal, B.Cu at (238.6, 81.0)
- added G***: LOGO, kbd:corne-logo-horizontal, F.Cu at (238.8, 81.0)
- added G***: LOGO, kbd:corne-logo-horizontal, B.Cu at (58.0, 80.9)
- added G***: LOGO, kbd:corne-logo-horizontal, F.Cu at (58.3, 80.9)
- added J1: MJ-4PP-9, kbd:MJ-4PP-9_1side, F.Cu at (144.1, 74.3)
- added J2: OLED, custom_kicad:OLED_1side, F.Cu at (130.9, 67.0)
- added J4: OLED, custom_kicad:OLED_1side, F.Cu at (165.8, 67.0)
- added LED1: WS2812B, LED_SMD:LED_WS2812B_PLCC4_5.0x5.0mm_P3.2mm, B.Cu at (47.7, 45.3)
- added LED10: YS-SK6812MINI-E, kbd:YS-SK6812MINI-E, B.Cu at (77.1, 23.9)
- added LED11: YS-SK6812MINI-E, kbd:YS-SK6812MINI-E, B.Cu at (96.1, 26.3)
- added LED12: YS-SK6812MINI-E, kbd:YS-SK6812MINI-E, B.Cu at (115.1, 28.7)
- added LED13: YS-SK6812MINI-E, kbd:YS-SK6812MINI-E, B.Cu at (20.1, 50.1)
- added LED14: YS-SK6812MINI-E, kbd:YS-SK6812MINI-E, B.Cu at (39.1, 50.1)
- added LED15: YS-SK6812MINI-E, kbd:YS-SK6812MINI-E, B.Cu at (58.1, 45.3)
- added LED16: YS-SK6812MINI-E, kbd:YS-SK6812MINI-E, B.Cu at (77.1, 42.9)
- added LED17: YS-SK6812MINI-E, kbd:YS-SK6812MINI-E, B.Cu at (96.1, 45.3)
- added LED18: YS-SK6812MINI-E, kbd:YS-SK6812MINI-E, B.Cu at (115.1, 47.7)
- added LED19: YS-SK6812MINI-E, kbd:YS-SK6812MINI-E, B.Cu at (20.1, 69.1)
- added LED2: WS2812B, LED_SMD:LED_WS2812B_PLCC4_5.0x5.0mm_P3.2mm, B.Cu at (68.9, 39.2)
- added LED20: YS-SK6812MINI-E, kbd:YS-SK6812MINI-E, B.Cu at (39.1, 69.1)
- added LED21: YS-SK6812MINI-E, kbd:YS-SK6812MINI-E, B.Cu at (58.1, 64.3)
- added LED22: YS-SK6812MINI-E, kbd:YS-SK6812MINI-E, B.Cu at (77.1, 61.9)
- added LED23: YS-SK6812MINI-E, kbd:YS-SK6812MINI-E, B.Cu at (96.1, 64.3)
- added LED24: YS-SK6812MINI-E, kbd:YS-SK6812MINI-E, B.Cu at (115.1, 66.7)
- added LED25: YS-SK6812MINI-E, kbd:YS-SK6812MINI-E, B.Cu at (86.6, 83.9)
- added LED26: YS-SK6812MINI-E, kbd:YS-SK6812MINI-E, B.Cu at (108.8, 86.9)
- added LED27: YS-SK6812MINI-E, kbd:YS-SK6812MINI-E, B.Cu at (134.0, 97.5)
- added LED28: WS2812B, LED_SMD:LED_WS2812B_PLCC4_5.0x5.0mm_P3.2mm, B.Cu at (250.6, 45.3)
- added LED29: WS2812B, LED_SMD:LED_WS2812B_PLCC4_5.0x5.0mm_P3.2mm, B.Cu at (227.7, 39.3)
- added LED3: WS2812B, LED_SMD:LED_WS2812B_PLCC4_5.0x5.0mm_P3.2mm, B.Cu at (105.8, 46.9)
- added LED30: WS2812B, LED_SMD:LED_WS2812B_PLCC4_5.0x5.0mm_P3.2mm, B.Cu at (191.0, 46.9)
- added LED31: WS2812B, LED_SMD:LED_WS2812B_PLCC4_5.0x5.0mm_P3.2mm, B.Cu at (250.6, 64.3)
- added LED32: WS2812B, LED_SMD:LED_WS2812B_PLCC4_5.0x5.0mm_P3.2mm, B.Cu at (218.1, 79.1)
- added LED33: WS2812B, LED_SMD:LED_WS2812B_PLCC4_5.0x5.0mm_P3.2mm, B.Cu at (178.6, 83.6)
- added LED34: YS-SK6812MINI-E, kbd:YS-SK6812MINI-E, B.Cu at (276.6, 31.1)
- added LED35: YS-SK6812MINI-E, kbd:YS-SK6812MINI-E, B.Cu at (257.6, 31.1)
- added LED36: YS-SK6812MINI-E, kbd:YS-SK6812MINI-E, B.Cu at (238.6, 26.3)
- added LED37: YS-SK6812MINI-E, kbd:YS-SK6812MINI-E, B.Cu at (219.6, 23.9)
- added LED38: YS-SK6812MINI-E, kbd:YS-SK6812MINI-E, B.Cu at (200.6, 26.3)
- added LED39: YS-SK6812MINI-E, kbd:YS-SK6812MINI-E, B.Cu at (181.6, 28.7)
- added LED4: WS2812B, LED_SMD:LED_WS2812B_PLCC4_5.0x5.0mm_P3.2mm, B.Cu at (48.3, 64.3)
- added LED40: YS-SK6812MINI-E, kbd:YS-SK6812MINI-E, B.Cu at (276.6, 50.1)
- added LED41: YS-SK6812MINI-E, kbd:YS-SK6812MINI-E, B.Cu at (257.6, 50.1)
- added LED42: YS-SK6812MINI-E, kbd:YS-SK6812MINI-E, B.Cu at (238.6, 45.3)
- added LED43: YS-SK6812MINI-E, kbd:YS-SK6812MINI-E, B.Cu at (219.6, 42.9)
- added LED44: YS-SK6812MINI-E, kbd:YS-SK6812MINI-E, B.Cu at (200.6, 45.3)
- added LED45: YS-SK6812MINI-E, kbd:YS-SK6812MINI-E, B.Cu at (181.6, 47.7)
- added LED46: YS-SK6812MINI-E, kbd:YS-SK6812MINI-E, B.Cu at (276.6, 69.1)
- added LED47: YS-SK6812MINI-E, kbd:YS-SK6812MINI-E, B.Cu at (257.6, 69.1)
- added LED48: YS-SK6812MINI-E, kbd:YS-SK6812MINI-E, B.Cu at (238.6, 64.3)
- added LED49: YS-SK6812MINI-E, kbd:YS-SK6812MINI-E, B.Cu at (219.6, 61.9)
- added LED5: WS2812B, LED_SMD:LED_WS2812B_PLCC4_5.0x5.0mm_P3.2mm, B.Cu at (78.8, 79.1)
- added LED50: YS-SK6812MINI-E, kbd:YS-SK6812MINI-E, B.Cu at (200.6, 64.3)
- added LED51: YS-SK6812MINI-E, kbd:YS-SK6812MINI-E, B.Cu at (181.6, 66.7)
- added LED52: YS-SK6812MINI-E, kbd:YS-SK6812MINI-E, B.Cu at (210.1, 83.9)
- added LED53: YS-SK6812MINI-E, kbd:YS-SK6812MINI-E, B.Cu at (187.9, 86.8)
- added LED54: YS-SK6812MINI-E, kbd:YS-SK6812MINI-E, B.Cu at (162.8, 97.5)
- added LED6: WS2812B, LED_SMD:LED_WS2812B_PLCC4_5.0x5.0mm_P3.2mm, B.Cu at (118.1, 83.6)
- added LED7: YS-SK6812MINI-E, kbd:YS-SK6812MINI-E, B.Cu at (20.1, 31.1)
- added LED8: YS-SK6812MINI-E, kbd:YS-SK6812MINI-E, B.Cu at (39.1, 31.1)
- added LED9: YS-SK6812MINI-E, kbd:YS-SK6812MINI-E, B.Cu at (58.1, 26.3)
- added REF**: Breakaway_Tabs, kbd:Breakaway_Tabs, B.Cu at (238.6, 21.9)
- added REF**: Breakaway_Tabs, kbd:Breakaway_Tabs, B.Cu at (200.7, 21.9)
- added REF**: Breakaway_Tabs, kbd:Breakaway_Tabs, B.Cu at (238.7, 83.2)
- added REF**: Breakaway_Tabs, kbd:Breakaway_Tabs, B.Cu at (276.7, 83.2)
- added REF**: Breakaway_Tabs, kbd:Breakaway_Tabs, F.Cu at (58.1, 83.2)
- added REF**: Breakaway_Tabs, kbd:Breakaway_Tabs, F.Cu at (20.2, 83.2)
- added REF**: Breakaway_Tabs, kbd:Breakaway_Tabs, F.Cu at (96.2, 21.9)
- added REF**: Breakaway_Tabs, kbd:Breakaway_Tabs, F.Cu at (58.2, 21.9)
- added RSW2: SW_PUSH, kbd:ResetSW_1side, F.Cu at (154.3, 66.5)
- added Ref**: Val**, kbd:M2_HOLE_v2, B.Cu at (168.9, 74.3)
- added Ref**: Val**, kbd:M2_HOLE_v2, F.Cu at (119.3, 89.1)
- added Ref**: Val**, kbd:M2_HOLE_v2, F.Cu at (72.8, 81.5)
- added Ref**: Val**, kbd:M2_HOLE_v2, F.Cu at (105.6, 41.8)
- added Ref**: Val**, kbd:M2_HOLE_v2, F.Cu at (27.5, 54.1)
- added Ref**: Val**, kbd:M2_HOLE_v2, F.Cu at (29.6, 45.3)
- added Ref**: Val**, kbd:M2_HOLE_v2, B.Cu at (269.2, 54.1)
- added Ref**: Val**, kbd:M2_HOLE_v2, B.Cu at (191.1, 41.8)
- added Ref**: Val**, kbd:M2_HOLE_v2, B.Cu at (267.1, 45.3)
- added Ref**: Val**, kbd:M2_HOLE_v2, B.Cu at (224.0, 81.5)
- added Ref**: Val**, kbd:M2_HOLE_v2, B.Cu at (154.4, 82.8)
- added Ref**: Val**, kbd:M2_HOLE_v2, B.Cu at (177.4, 89.1)
- added Ref**: Val**, kbd:M2_HOLE_v2, F.Cu at (142.3, 82.8)
- added Ref**: Val**, kbd:M2_HOLE_v2, F.Cu at (127.9, 74.3)
- added SW22: SW_PUSH, custom_kicad:PG1350_socket_clean, F.Cu at (276.6, 35.8)
- added SW23: SW_PUSH, custom_kicad:PG1350_socket_clean, F.Cu at (257.6, 35.8)
- added SW24: SW_PUSH, custom_kicad:PG1350_socket_clean, F.Cu at (238.6, 31.0)
- added SW25: SW_PUSH, custom_kicad:PG1350_socket_clean, F.Cu at (219.6, 28.6)
- added SW26: SW_PUSH, custom_kicad:PG1350_socket_clean, F.Cu at (200.6, 31.0)
- added SW27: SW_PUSH, custom_kicad:PG1350_socket_clean, F.Cu at (181.6, 33.4)
- added SW28: SW_PUSH, custom_kicad:PG1350_socket_clean, F.Cu at (276.6, 54.8)
- added SW29: SW_PUSH, custom_kicad:PG1350_socket_clean, F.Cu at (257.6, 54.8)
- added SW30: SW_PUSH, custom_kicad:PG1350_socket_clean, F.Cu at (238.6, 50.0)
- added SW31: SW_PUSH, custom_kicad:PG1350_socket_clean, F.Cu at (219.6, 47.6)
- added SW32: SW_PUSH, custom_kicad:PG1350_socket_clean, F.Cu at (200.6, 50.0)
- added SW33: SW_PUSH, custom_kicad:PG1350_socket_clean, F.Cu at (181.6, 52.4)
- added SW34: SW_PUSH, custom_kicad:PG1350_socket_clean, F.Cu at (276.6, 73.8)
- added SW35: SW_PUSH, custom_kicad:PG1350_socket_clean, F.Cu at (257.6, 73.8)
- added SW36: SW_PUSH, custom_kicad:PG1350_socket_clean, F.Cu at (238.6, 69.0)
- added SW37: SW_PUSH, custom_kicad:PG1350_socket_clean, F.Cu at (219.6, 66.7)
- added SW38: SW_PUSH, custom_kicad:PG1350_socket_clean, F.Cu at (200.6, 69.0)
- added SW39: SW_PUSH, custom_kicad:PG1350_socket_clean, F.Cu at (181.6, 71.4)
- added SW40: SW_PUSH, custom_kicad:PG1350_socket_clean, F.Cu at (210.1, 88.7)
- added SW41: SW_PUSH, custom_kicad:PG1350_socket_clean, F.Cu at (189.1, 91.4)
- added SW42: SW_PUSH, custom_kicad:PG1350_socket_clean, F.Cu at (166.9, 95.2)
- added U2: ProMicro, custom_kicad:ProMicro_v3, F.Cu at (162.0, 46.4)
- D1, D10, D11, D12, D13, D14, D15, D16, D17, D18, D19, D2, D20, D21, D3, D4, D5, D6, D7, D8, D9: footprint kbd:D3_SMD -> kbd:D3_SMD_v2; moved to B.Cu
- J3: value LED -> MJ-4PP-9; footprint kbd:StripLED_rev -> kbd:MJ-4PP-9_1side
- RSW1: value Reset -> SW_PUSH; footprint kbd:ResetSW -> kbd:ResetSW_1side
- SW1, SW10, SW11, SW12, SW13, SW14, SW15, SW16, SW17, SW18, SW19, SW2, SW20, SW3, SW4, SW5, SW6, SW7, SW8, SW9: footprint kbd:Choc_Hotswap -> custom_kicad:PG1350_socket_clean
- SW21: footprint kbd:Choc_Hotswap_1.5u -> custom_kicad:PG1350_socket_clean
- U1: footprint kbd:ProMicro_v2 -> custom_kicad:ProMicro_v3
- moved D19 66.1 mm to (76.2, 87.6), turned to 90 degrees
- moved SW1 64.8 mm to (20.1, 35.8), turned to 0 degrees
- moved SW10 64.8 mm to (77.1, 47.7), turned to 0 degrees
- moved SW11 64.8 mm to (96.1, 50.0), turned to 0 degrees
- moved SW12 64.8 mm to (115.1, 52.4), turned to 0 degrees
- moved SW13 64.8 mm to (20.1, 73.8), turned to 0 degrees
- moved SW14 64.8 mm to (39.1, 73.8), turned to 0 degrees
- moved SW15 64.8 mm to (58.1, 69.0), turned to 0 degrees
- moved SW16 64.8 mm to (77.1, 66.7), turned to 0 degrees
- moved SW17 64.8 mm to (96.1, 69.0), turned to 0 degrees
- moved SW18 64.8 mm to (115.1, 71.4), turned to 0 degrees
- moved SW19 64.8 mm to (86.6, 88.7), turned to 0 degrees
- moved SW2 64.8 mm to (39.1, 35.8), turned to 0 degrees
- moved SW20 64.8 mm to (107.6, 91.4), turned to 345 degrees
- moved SW21 64.8 mm to (129.9, 95.2)
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Routing:
- net VDD: track 0.00 -> 550.3 mm, vias 0 -> 42
- net GNDA: track 0.00 -> 546.2 mm, vias 0 -> 32
- net VCC: track 786.4 -> 520.4 mm, vias 30 -> 41
- net GND: track 816.7 -> 586.5 mm, vias 59 -> 38
- net col0_r: track 0.00 -> 177.9 mm, vias 0 -> 7
- net row2_r: track 0.00 -> 156.6 mm, vias 0 -> 6
- net col1_r: track 0.00 -> 155.4 mm, vias 0 -> 5
- net col3_r: track 0.00 -> 147.8 mm, vias 0 -> 8
- net row0_r: track 0.00 -> 144.8 mm, vias 0 -> 6
- net row1_r: track 0.00 -> 140.6 mm, vias 0 -> 6
- net col2_r: track 0.00 -> 132.4 mm, vias 0 -> 5
- net col4_r: track 0.00 -> 125.5 mm, vias 0 -> 6
- net col5: track 188.2 -> 70.3 mm, vias 10 -> 4
- net col1: track 232.6 -> 130.5 mm, vias 7 -> 3
- net col0: track 255.1 -> 154.0 mm, vias 12 -> 3
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- removed copper zone on B.Cu, net GND
- removed copper zone on F.Cu, net GND
Other:
- board size 133.8 x 91.4 mm -> 275.5 x 105.6 mm
- net class thick added: clearance 0.2, trace_width 0.5, via_dia 0.6, via_drill 0.4
- board text added: "Corne Chocolate v3.0 by Boardsource PCB Designed by foostan"
- board text removed: "Corne Chocolate v2.1 PCB designed by foostan"
- board text removed: "GND"
- board text removed: "LED"
- board text removed: "OLED"
- board text removed: "VCC"

Commit message: Update corne-chocolate to KiCad 6.0.8
Other:
- net class Default removed
- net class thick removed
